File: validation/BlackPill_validation.kicad_pcb (KiCad board)
At the start: 2 copper layers, 70 x 40 mm, 1 part, among them U1 WeAct_BlackPill_MiniF4_STM32F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

Commit message: 3d images
Other:
- board text added: "ASTRA CanSat"
- board text removed: "ASTRA CanSat - footprint + official STEP validation"
